File: Manual-Traffic-Signal-System.brd (EAGLE design)
At the start: 68.6 x 53.3 mm, 9 parts

Commit message: Design updated for two buttons
Parts:
- removed Dled_green, Dled_yellow: (no value), AUTODESK_CIRCUITS_BREADBOARD:LED5MM
- removed Son_off: (no value), AUTODESK_CIRCUITS_BREADBOARD:TL1105
- added D10, D11, D12, D13, D2, D3, D4, D5, D6, D8, D9: (no value), AUTODESK_CIRCUITS_BREADBOARD:LED5MM
- added R10, R11, R12, R13, R14, R15, R5, R7, R8, R9: 220‎Ω, AUTODESK_CIRCUITS_BREADBOARD:0207/10
- added S2, S3: (no value), AUTODESK_CIRCUITS_BREADBOARD:TL1105
- R2: value 220‎Ω -> 1k‎Ω
- moved R2 279.4 mm to (5.00, 353.0)
- moved R4 254.0 mm to (5.00, 365.7)
- moved R3 50.8 mm to (5.00, 35.5)
- renumbered Dled_red to D1, R1 to R6
Connections:
- new net N$12: D6.A, Uarduino.6
- new net N$13: D10.K, R10.1
- new net N$14: D10.A, Uarduino.9
- new net N$15: D8.K, R12.1
- new net N$16: D8.A, Uarduino.11
- new net N$17: D11.K, R13.2
- new net N$18: D11.A, Uarduino.A0
- new net N$19: D12.K, R14.2
- new net N$20: D12.A, Uarduino.A1
- new net N$21: D9.K, R15.2
- new net N$22: D9.A, Uarduino.2
- new net N$23: D13.K, R11.1
- new net N$24: D13.A, Uarduino.10
- new net N$25: S2.4
- new net N$26: R4.1, S2.2, Uarduino.12
- new net N$27: S2.1
- new net N$28: S3.4
- new net N$29: R2.1, S3.2, Uarduino.A2
- new net N$30: S3.1
- new net N$31: S2.3, S3.3, Uarduino.5V
- new net N$32: R10.2, R11.2, R12.2, R13.1, R14.1, R15.1, R2.2, R3.1, R4.2, R5.1, R6.1, R7.2, R8.2, R9.2, Uarduino.GND
- net N$1: now also D2.K, R5.2; no longer Dled_green.K, R6.2
- net N$10: now also D4.A, Uarduino.8; no longer Son_off.4
- net N$11: now also D5.A, Uarduino.7; no longer Son_off.3
- net N$2: now also D2.A, Uarduino.5; no longer D1.K, R2.2
- net N$3: now also D3.K, R6.2; no longer Dled_yellow.K, R3.2
- net N$4: now also D3.A, Uarduino.4; no longer D1.A, Uarduino.11
- net N$5: now also D1.K, R3.2; no longer Dled_green.A, Uarduino.12
- net N$6: now also D1.A, Uarduino.3; no longer Dled_yellow.A, Uarduino.13
- net N$7: now also D6.K, R7.1; no longer R2.1, R3.1, R4.1, R6.1, Uarduino.GND
- net N$8: now also D5.K, R8.1; no longer Son_off.2, Uarduino.3.3V
- net N$9: now also D4.K, R9.1; no longer R4.2, Son_off.1, Uarduino.7
